File: tikk-hw.kicad_pcb (KiCad board)
At the start: 4 copper layers, 18.1 x 39 mm, 116 parts, among them P6 ZX-SH1.0-4PWT, SW1 TS24CA, SW2 TS24CA, U1 IS31FL3731-QFLS2-TR, U2 LIS2DH12TR, U4 CP6208DTR(XBLW), U5 TMP102AIDRLR

Commit message: initial placements all finished
Parts:
- removed the LED1 at (169.1, 110.5)
- removed the LED1 at (169.2, 112.3)
- removed the LED1 at (169.0, 97.8)
- removed the LED1 at (169.0, 108.7)
- removed the LED1 at (169.2, 114.2)
- removed the LED1 at (169.0, 99.6)
- removed the LED1 at (169.1, 106.9)
- removed the LED1 at (169.1, 101.4)
- removed the LED1 at (169.1, 105.1)
- removed the LED1 at (169.0, 96.0)
- removed the LED1 at (168.9, 94.1)
- removed the LED1 at (169.0, 103.3)
- removed the LED1 at (168.9, 92.2)
- removed the LED1 at (169.2, 116.0)
- removed the LED2 at (167.3, 99.6)
- removed the LED2 at (167.4, 103.4)
- removed the LED2 at (167.3, 97.8)
- removed the LED2 at (167.5, 110.7)
- removed the LED2 at (167.4, 106.9)
- removed the LED2 at (167.4, 105.2)
- removed the LED2 at (167.2, 94.1)
- removed the LED2 at (167.5, 114.2)
- removed the LED2 at (167.3, 101.5)
- removed the LED2 at (167.3, 96.0)
- removed the LED2 at (167.5, 116.1)
- removed the LED2 at (169.2, 117.8)
- removed the LED2 at (167.4, 108.8)
- removed the LED2 at (167.6, 117.9)
- removed the LED2 at (167.5, 112.5)
- removed the LED2 at (167.2, 92.2)
- removed the LED3 at (165.7, 106.9)
- removed the LED3 at (165.8, 110.7)
- removed the LED3 at (165.7, 103.3)
- removed the LED3 at (165.6, 101.5)
- removed the LED3 at (165.7, 105.2)
- removed the LED3 at (165.5, 94.1)
- removed the LED3 at (165.7, 108.8)
- removed the LED3 at (165.6, 96.0)
- removed the LED3 at (165.8, 116.0)
- removed the LED3 at (165.9, 117.9)
- removed the LED3 at (165.8, 114.2)
- removed the LED3 at (165.5, 92.2)
- removed the LED3 at (165.6, 99.6)
- removed the LED3 at (165.6, 97.8)
- removed the LED3 at (165.8, 112.5)
- removed the LED4 at (164.1, 103.4)
- removed the LED4 at (164.2, 110.7)
- removed the LED4 at (164.0, 101.5)
- removed the LED4 at (164.0, 97.8)
- removed the LED4 at (164.0, 96.0)
- removed the LED4 at (164.1, 107.0)
- removed the LED4 at (164.2, 116.1)
- removed the LED4 at (164.2, 112.5)
- removed the LED4 at (163.9, 92.3)
- removed the LED4 at (164.0, 99.7)
- removed the LED4 at (164.2, 118.0)
- removed the LED4 at (164.2, 114.2)
- removed the LED4 at (163.9, 94.2)
- removed the LED4 at (164.1, 105.2)
- removed the LED4 at (164.1, 108.8)
- removed the LED5 at (162.3, 97.8)
- removed the LED5 at (162.4, 108.8)
- removed the LED5 at (162.3, 101.5)
- removed the LED5 at (162.5, 116.1)
- removed the LED5 at (162.4, 110.7)
- removed the LED5 at (162.4, 112.5)
- removed the LED5 at (162.6, 118.0)
- removed the LED5 at (162.2, 92.3)
- removed the LED5 at (162.3, 103.4)
- removed the LED5 at (162.3, 99.7)
- removed the LED5 at (162.3, 96.0)
- removed the LED5 at (162.5, 114.2)
- removed the LED5 at (162.4, 107.0)
- removed the LED5 at (162.3, 105.2)
- removed the LED5 at (162.2, 94.2)
- removed the LED6 at (160.6, 103.4)
- removed the LED6 at (160.7, 116.1)
- removed the LED6 at (160.5, 101.5)
- removed the LED6 at (160.8, 117.9)
- removed the LED6 at (160.5, 99.6)
- removed the LED6 at (160.6, 108.8)
- removed the LED6 at (160.6, 106.9)
- removed the LED6 at (160.7, 110.7)
- removed the LED6 at (160.5, 97.8)
- removed the LED6 at (160.4, 92.2)
- removed the LED6 at (160.7, 112.5)
- removed the LED6 at (160.7, 114.2)
- removed the LED6 at (160.4, 94.1)
- removed the LED6 at (160.6, 105.2)
- removed the LED6 at (160.5, 96.0)
- removed the LED7 at (159.0, 114.2)
- removed the LED7 at (159.0, 112.5)
- removed the LED7 at (158.9, 108.8)
- removed the LED7 at (158.9, 103.4)
- removed the LED7 at (158.9, 106.9)
- removed the LED7 at (158.8, 101.5)
- removed the LED7 at (158.8, 96.0)
- removed the LED7 at (158.9, 105.2)
- removed the LED7 at (158.8, 97.8)
- removed the LED7 at (158.7, 94.1)
- removed the LED7 at (159.0, 110.7)
- removed the LED7 at (158.7, 92.2)
- removed the LED7 at (158.8, 99.6)
- removed the LED7 at (159.0, 116.1)
- removed the LED7 at (159.1, 117.9)
- added J1: 51281-0598, easyeda2kicad:512810598, F.Cu at (163.7, 122.2)
- added LED1: F.0402.00003/P2-0402R1TS2-045T-001, easyeda2kicad:LED0402-RD, B.Cu at (169.3, 92.2)
- added LED10: F.0402.00003/P2-0402R1TS2-045T-001, easyeda2kicad:LED0402-RD, B.Cu at (165.7, 94.0)
- added LED100: F.0402.00003/P2-0402R1TS2-045T-001, easyeda2kicad:LED0402-RD, B.Cu at (167.5, 110.2)
- added LED101: F.0402.00003/P2-0402R1TS2-045T-001, easyeda2kicad:LED0402-RD, B.Cu at (165.7, 110.2)
- added LED102: F.0402.00003/P2-0402R1TS2-045T-001, easyeda2kicad:LED0402-RD, B.Cu at (163.9, 110.2)
- added LED103: F.0402.00003/P2-0402R1TS2-045T-001, easyeda2kicad:LED0402-RD, B.Cu at (162.1, 110.2)
- added LED104: F.0402.00003/P2-0402R1TS2-045T-001, easyeda2kicad:LED0402-RD, B.Cu at (160.3, 110.2)
- added LED105: F.0402.00003/P2-0402R1TS2-045T-001, easyeda2kicad:LED0402-RD, B.Cu at (158.5, 110.2)
- added LED11: F.0402.00003/P2-0402R1TS2-045T-001, easyeda2kicad:LED0402-RD, B.Cu at (163.9, 94.0)
- added LED12: F.0402.00003/P2-0402R1TS2-045T-001, easyeda2kicad:LED0402-RD, B.Cu at (162.1, 94.0)
- added LED13: F.0402.00003/P2-0402R1TS2-045T-001, easyeda2kicad:LED0402-RD, B.Cu at (160.3, 94.0)
- added LED14: F.0402.00003/P2-0402R1TS2-045T-001, easyeda2kicad:LED0402-RD, B.Cu at (158.5, 94.0)
- added LED15: F.0402.00003/P2-0402R1TS2-045T-001, easyeda2kicad:LED0402-RD, B.Cu at (169.3, 95.8)
- added LED16: F.0402.00003/P2-0402R1TS2-045T-001, easyeda2kicad:LED0402-RD, B.Cu at (167.5, 95.8)
- added LED17: F.0402.00003/P2-0402R1TS2-045T-001, easyeda2kicad:LED0402-RD, B.Cu at (165.7, 95.8)
- added LED18: F.0402.00003/P2-0402R1TS2-045T-001, easyeda2kicad:LED0402-RD, B.Cu at (163.9, 95.8)
- added LED19: F.0402.00003/P2-0402R1TS2-045T-001, easyeda2kicad:LED0402-RD, B.Cu at (162.1, 95.8)
- added LED2: F.0402.00003/P2-0402R1TS2-045T-001, easyeda2kicad:LED0402-RD, B.Cu at (167.5, 92.2)
- added LED20: F.0402.00003/P2-0402R1TS2-045T-001, easyeda2kicad:LED0402-RD, B.Cu at (160.3, 95.8)
- added LED21: F.0402.00003/P2-0402R1TS2-045T-001, easyeda2kicad:LED0402-RD, B.Cu at (158.5, 95.8)
- added LED22: F.0402.00003/P2-0402R1TS2-045T-001, easyeda2kicad:LED0402-RD, B.Cu at (169.3, 97.6)
- added LED23: F.0402.00003/P2-0402R1TS2-045T-001, easyeda2kicad:LED0402-RD, B.Cu at (167.5, 97.6)
- added LED24: F.0402.00003/P2-0402R1TS2-045T-001, easyeda2kicad:LED0402-RD, B.Cu at (165.7, 97.6)
- added LED25: F.0402.00003/P2-0402R1TS2-045T-001, easyeda2kicad:LED0402-RD, B.Cu at (163.9, 97.6)
- added LED26: F.0402.00003/P2-0402R1TS2-045T-001, easyeda2kicad:LED0402-RD, B.Cu at (162.1, 97.6)
- added LED27: F.0402.00003/P2-0402R1TS2-045T-001, easyeda2kicad:LED0402-RD, B.Cu at (160.3, 97.6)
- added LED28: F.0402.00003/P2-0402R1TS2-045T-001, easyeda2kicad:LED0402-RD, B.Cu at (158.5, 97.6)
- added LED29: F.0402.00003/P2-0402R1TS2-045T-001, easyeda2kicad:LED0402-RD, B.Cu at (169.3, 99.4)
- added LED3: F.0402.00003/P2-0402R1TS2-045T-001, easyeda2kicad:LED0402-RD, B.Cu at (165.7, 92.2)
- added LED30: F.0402.00003/P2-0402R1TS2-045T-001, easyeda2kicad:LED0402-RD, B.Cu at (167.4, 99.4)
- added LED31: F.0402.00003/P2-0402R1TS2-045T-001, easyeda2kicad:LED0402-RD, B.Cu at (165.7, 99.4)
- added LED32: F.0402.00003/P2-0402R1TS2-045T-001, easyeda2kicad:LED0402-RD, B.Cu at (163.9, 99.4)
- added LED33: F.0402.00003/P2-0402R1TS2-045T-001, easyeda2kicad:LED0402-RD, B.Cu at (162.1, 99.4)
- added LED34: F.0402.00003/P2-0402R1TS2-045T-001, easyeda2kicad:LED0402-RD, B.Cu at (160.3, 99.4)
- added LED35: F.0402.00003/P2-0402R1TS2-045T-001, easyeda2kicad:LED0402-RD, B.Cu at (158.5, 99.4)
- added LED36: F.0402.00003/P2-0402R1TS2-045T-001, easyeda2kicad:LED0402-RD, B.Cu at (169.3, 108.4)
- added LED37: F.0402.00003/P2-0402R1TS2-045T-001, easyeda2kicad:LED0402-RD, B.Cu at (167.5, 108.4)
- added LED38: F.0402.00003/P2-0402R1TS2-045T-001, easyeda2kicad:LED0402-RD, B.Cu at (165.7, 108.4)
- added LED39: F.0402.00003/P2-0402R1TS2-045T-001, easyeda2kicad:LED0402-RD, B.Cu at (163.9, 108.4)
- added LED4: F.0402.00003/P2-0402R1TS2-045T-001, easyeda2kicad:LED0402-RD, B.Cu at (163.9, 92.2)
- added LED40: F.0402.00003/P2-0402R1TS2-045T-001, easyeda2kicad:LED0402-RD, B.Cu at (162.1, 108.4)
- added LED41: F.0402.00003/P2-0402R1TS2-045T-001, easyeda2kicad:LED0402-RD, B.Cu at (160.3, 108.4)
- added LED42: F.0402.00003/P2-0402R1TS2-045T-001, easyeda2kicad:LED0402-RD, B.Cu at (158.5, 108.4)
- added LED43: F.0402.00003/P2-0402R1TS2-045T-001, easyeda2kicad:LED0402-RD, B.Cu at (169.3, 106.6)
- added LED44: F.0402.00003/P2-0402R1TS2-045T-001, easyeda2kicad:LED0402-RD, B.Cu at (167.5, 106.6)
- added LED45: F.0402.00003/P2-0402R1TS2-045T-001, easyeda2kicad:LED0402-RD, B.Cu at (165.7, 106.6)
- added LED46: F.0402.00003/P2-0402R1TS2-045T-001, easyeda2kicad:LED0402-RD, B.Cu at (163.9, 106.6)
- added LED47: F.0402.00003/P2-0402R1TS2-045T-001, easyeda2kicad:LED0402-RD, B.Cu at (162.1, 106.6)
- added LED48: F.0402.00003/P2-0402R1TS2-045T-001, easyeda2kicad:LED0402-RD, B.Cu at (160.3, 106.6)
- added LED49: F.0402.00003/P2-0402R1TS2-045T-001, easyeda2kicad:LED0402-RD, B.Cu at (158.5, 106.6)
- added LED5: F.0402.00003/P2-0402R1TS2-045T-001, easyeda2kicad:LED0402-RD, B.Cu at (162.1, 92.2)
- added LED50: F.0402.00003/P2-0402R1TS2-045T-001, easyeda2kicad:LED0402-RD, B.Cu at (169.3, 104.8)
- added LED51: F.0402.00003/P2-0402R1TS2-045T-001, easyeda2kicad:LED0402-RD, B.Cu at (167.5, 104.8)
- added LED52: F.0402.00003/P2-0402R1TS2-045T-001, easyeda2kicad:LED0402-RD, B.Cu at (165.7, 104.8)
- added LED53: F.0402.00003/P2-0402R1TS2-045T-001, easyeda2kicad:LED0402-RD, B.Cu at (163.9, 104.8)
- added LED54: F.0402.00003/P2-0402R1TS2-045T-001, easyeda2kicad:LED0402-RD, B.Cu at (162.1, 104.8)
- added LED55: F.0402.00003/P2-0402R1TS2-045T-001, easyeda2kicad:LED0402-RD, B.Cu at (160.3, 104.8)
- added LED56: F.0402.00003/P2-0402R1TS2-045T-001, easyeda2kicad:LED0402-RD, B.Cu at (158.5, 104.8)
- added LED57: F.0402.00003/P2-0402R1TS2-045T-001, easyeda2kicad:LED0402-RD, B.Cu at (169.3, 103.0)
- added LED58: F.0402.00003/P2-0402R1TS2-045T-001, easyeda2kicad:LED0402-RD, B.Cu at (167.5, 103.0)
- added LED59: F.0402.00003/P2-0402R1TS2-045T-001, easyeda2kicad:LED0402-RD, B.Cu at (165.7, 103.0)
- added LED6: F.0402.00003/P2-0402R1TS2-045T-001, easyeda2kicad:LED0402-RD, B.Cu at (160.3, 92.2)
- added LED60: F.0402.00003/P2-0402R1TS2-045T-001, easyeda2kicad:LED0402-RD, B.Cu at (163.9, 103.0)
- added LED61: F.0402.00003/P2-0402R1TS2-045T-001, easyeda2kicad:LED0402-RD, B.Cu at (162.1, 103.0)
- added LED62: F.0402.00003/P2-0402R1TS2-045T-001, easyeda2kicad:LED0402-RD, B.Cu at (160.3, 103.0)
- added LED63: F.0402.00003/P2-0402R1TS2-045T-001, easyeda2kicad:LED0402-RD, B.Cu at (158.5, 103.0)
- added LED64: F.0402.00003/P2-0402R1TS2-045T-001, easyeda2kicad:LED0402-RD, B.Cu at (169.3, 101.2)
- added LED65: F.0402.00003/P2-0402R1TS2-045T-001, easyeda2kicad:LED0402-RD, B.Cu at (167.4, 101.2)
- added LED66: F.0402.00003/P2-0402R1TS2-045T-001, easyeda2kicad:LED0402-RD, B.Cu at (165.7, 101.2)
- added LED67: F.0402.00003/P2-0402R1TS2-045T-001, easyeda2kicad:LED0402-RD, B.Cu at (163.9, 101.2)
- added LED68: F.0402.00003/P2-0402R1TS2-045T-001, easyeda2kicad:LED0402-RD, B.Cu at (162.1, 101.2)
- added LED69: F.0402.00003/P2-0402R1TS2-045T-001, easyeda2kicad:LED0402-RD, B.Cu at (160.3, 101.2)
- added LED7: F.0402.00003/P2-0402R1TS2-045T-001, easyeda2kicad:LED0402-RD, B.Cu at (158.5, 92.2)
- added LED70: F.0402.00003/P2-0402R1TS2-045T-001, easyeda2kicad:LED0402-RD, B.Cu at (158.5, 101.2)
- added LED71: F.0402.00003/P2-0402R1TS2-045T-001, easyeda2kicad:LED0402-RD, B.Cu at (169.3, 117.4)
- added LED72: F.0402.00003/P2-0402R1TS2-045T-001, easyeda2kicad:LED0402-RD, B.Cu at (167.5, 117.4)
- added LED73: F.0402.00003/P2-0402R1TS2-045T-001, easyeda2kicad:LED0402-RD, B.Cu at (165.7, 117.4)
- added LED74: F.0402.00003/P2-0402R1TS2-045T-001, easyeda2kicad:LED0402-RD, B.Cu at (163.9, 117.4)
- added LED75: F.0402.00003/P2-0402R1TS2-045T-001, easyeda2kicad:LED0402-RD, B.Cu at (162.1, 117.4)
- added LED76: F.0402.00003/P2-0402R1TS2-045T-001, easyeda2kicad:LED0402-RD, B.Cu at (160.3, 117.4)
- added LED77: F.0402.00003/P2-0402R1TS2-045T-001, easyeda2kicad:LED0402-RD, B.Cu at (158.5, 117.4)
- added LED78: F.0402.00003/P2-0402R1TS2-045T-001, easyeda2kicad:LED0402-RD, B.Cu at (169.3, 115.6)
- added LED79: F.0402.00003/P2-0402R1TS2-045T-001, easyeda2kicad:LED0402-RD, B.Cu at (167.5, 115.6)
- added LED8: F.0402.00003/P2-0402R1TS2-045T-001, easyeda2kicad:LED0402-RD, B.Cu at (169.3, 94.0)
- added LED80: F.0402.00003/P2-0402R1TS2-045T-001, easyeda2kicad:LED0402-RD, B.Cu at (165.7, 115.6)
- added LED81: F.0402.00003/P2-0402R1TS2-045T-001, easyeda2kicad:LED0402-RD, B.Cu at (163.9, 115.6)
- added LED82: F.0402.00003/P2-0402R1TS2-045T-001, easyeda2kicad:LED0402-RD, B.Cu at (162.1, 115.6)
- added LED83: F.0402.00003/P2-0402R1TS2-045T-001, easyeda2kicad:LED0402-RD, B.Cu at (160.3, 115.6)
- added LED84: F.0402.00003/P2-0402R1TS2-045T-001, easyeda2kicad:LED0402-RD, B.Cu at (158.5, 115.6)
- added LED85: F.0402.00003/P2-0402R1TS2-045T-001, easyeda2kicad:LED0402-RD, B.Cu at (169.3, 113.8)
- added LED86: F.0402.00003/P2-0402R1TS2-045T-001, easyeda2kicad:LED0402-RD, B.Cu at (167.5, 113.8)
- added LED87: F.0402.00003/P2-0402R1TS2-045T-001, easyeda2kicad:LED0402-RD, B.Cu at (165.7, 113.8)
- added LED88: F.0402.00003/P2-0402R1TS2-045T-001, easyeda2kicad:LED0402-RD, B.Cu at (163.9, 113.8)
- added LED89: F.0402.00003/P2-0402R1TS2-045T-001, easyeda2kicad:LED0402-RD, B.Cu at (162.1, 113.8)
- added LED9: F.0402.00003/P2-0402R1TS2-045T-001, easyeda2kicad:LED0402-RD, B.Cu at (167.5, 94.0)
- added LED90: F.0402.00003/P2-0402R1TS2-045T-001, easyeda2kicad:LED0402-RD, B.Cu at (160.3, 113.8)
- added LED91: F.0402.00003/P2-0402R1TS2-045T-001, easyeda2kicad:LED0402-RD, B.Cu at (158.5, 113.8)
- added LED92: F.0402.00003/P2-0402R1TS2-045T-001, easyeda2kicad:LED0402-RD, B.Cu at (169.3, 112.0)
- added LED93: F.0402.00003/P2-0402R1TS2-045T-001, easyeda2kicad:LED0402-RD, B.Cu at (167.5, 112.0)
- added LED94: F.0402.00003/P2-0402R1TS2-045T-001, easyeda2kicad:LED0402-RD, B.Cu at (165.7, 112.0)
- added LED95: F.0402.00003/P2-0402R1TS2-045T-001, easyeda2kicad:LED0402-RD, B.Cu at (163.9, 112.0)
- added LED96: F.0402.00003/P2-0402R1TS2-045T-001, easyeda2kicad:LED0402-RD, B.Cu at (162.1, 112.0)
- added LED97: F.0402.00003/P2-0402R1TS2-045T-001, easyeda2kicad:LED0402-RD, B.Cu at (160.3, 112.0)
- added LED98: F.0402.00003/P2-0402R1TS2-045T-001, easyeda2kicad:LED0402-RD, B.Cu at (158.5, 112.0)
- added LED99: F.0402.00003/P2-0402R1TS2-045T-001, easyeda2kicad:LED0402-RD, B.Cu at (169.3, 110.2)
- added R1: 100K, Resistor_SMD:R_0402_1005Metric, F.Cu at (168.3, 100.4)
- added R1: 100K, Resistor_SMD:R_0402_1005Metric, F.Cu at (158.2, 100.4)
- added R2: 100K, Resistor_SMD:R_0402_1005Metric, F.Cu at (169.3, 100.4)
- added TP1: NC1, TestPoint:TestPoint_Pad_1.0x1.0mm, F.Cu at (164.6, 117.5)
- added TP2: NFC1, TestPoint:TestPoint_Pad_1.0x1.0mm, B.Cu at (167.9, 120.1)
- added TP3: NC2, TestPoint:TestPoint_Pad_1.0x1.0mm, F.Cu at (169.2, 117.5)
- added TP4: NC3, TestPoint:TestPoint_Pad_1.0x1.0mm, F.Cu at (166.9, 117.5)
- added TP5: NFC2, TestPoint:TestPoint_Pad_1.0x1.0mm, B.Cu at (169.9, 120.1)
- added TP6: SWCLK, TestPoint:TestPoint_THTPad_1.0x1.0mm_Drill0.5mm, F.Cu at (160.0, 120.1)
- added TP7: SWDIO, TestPoint:TestPoint_THTPad_1.0x1.0mm_Drill0.5mm, F.Cu at (158.4, 120.1)
- added U6: CP6208DTR(XBLW), easyeda2kicad:SOP-8_L4.9-W3.9-P1.27-LS6.0-BL, F.Cu at (160.9, 94.8)
- H1, H2, H3, P6, SW1, SW2: moved to B.Cu
- U1, U2, U4, U5: moved to F.Cu
- U3: renamed from U4; value CP6208DTR(XBLW) -> Tenstar nRF52840
- moved SW1 35.3 mm to (157.6, 122.6)
- moved SW2 35.3 mm to (169.9, 122.6)
- moved H1 35.1 mm to (170.4, 87.4)
- moved H2 35.1 mm to (156.9, 87.4)
- moved P6 32.6 mm to (163.8, 121.2)
- moved H3 30.4 mm to (163.7, 89.7)
- moved U4 19.5 mm to (166.9, 94.8)
- moved U1 15.8 mm to (163.9, 112.4), turned to 0 degrees
- moved U2 11.9 mm to (163.7, 106.2), turned to 0 degrees
- moved U5 3.89 mm to (168.9, 121.1)
Connections:
- H3 pad 1: unconnected-(H3-Pad1) -> Net-(U6-Bout)
- H3 pad 2: unconnected-(H3-Pad2) -> Net-(U6-Aout)
- H3 pad 3: unconnected-(H3-Pad3) -> Net-(U4-Bout)
- H3 pad 4: unconnected-(H3-Pad4) -> Net-(U4-Aout)
- SW1 pad 3: unconnected-(SW1-Pad3) -> GND
- SW1 pad 4: unconnected-(SW1-Pad4) -> RESET
- U3 pad 1: unconnected-(U4-Vcc-Pad1) -> VBAT
- U3 pad 10: (no net) -> /P1.11
- U3 pad 11: (no net) -> /P0.10
- U3 pad 12: (no net) -> /P0.09
- U3 pad 13: (no net) -> MOTOR1-A
- U3 pad 14: (no net) -> MOTOR1-B
- U3 pad 15: (no net) -> GND
- U3 pad 16: (no net) -> GND
- U3 pad 17: (no net) -> MOTOR2-A
- U3 pad 18: (no net) -> MOTOR2-B
- U3 pad 19: (no net) -> /P0.22
- U3 pad 2: unconnected-(U4-Bout-Pad2) -> GND
- U3 pad 20: (no net) -> /P0.24
- U3 pad 21: (no net) -> /P1.00
- U3 pad 22: (no net) -> /P0.13
- U3 pad 23: (no net) -> SCL
- U3 pad 24: (no net) -> SDA
- U3 pad 3: unconnected-(U4-Aout-Pad3) -> RESET
- U3 pad 4: unconnected-(U4-GND-Pad4) -> EXT_VCC
- U3 pad 5: unconnected-(U4-Bin-Pad5) -> BATTERY-V
- U3 pad 6: unconnected-(U4-NC-Pad6) -> /P0.29
- U3 pad 7: unconnected-(U4-GND-Pad7) -> /P0.02
- U3 pad 8: unconnected-(U4-Ain-Pad8) -> /P1.15
- U3 pad 9: (no net) -> /P1.13
- U4 pad 2: unconnected-(U4-Bout-Pad2) -> Net-(U4-Bout)
- U4 pad 3: unconnected-(U4-Aout-Pad3) -> Net-(U4-Aout)
- U4 pad 5: unconnected-(U4-Bin-Pad5) -> MOTOR2-B
- U4 pad 8: unconnected-(U4-Ain-Pad8) -> MOTOR2-A
- U5 pad 1: unconnected-(U5-SCL-Pad1) -> SCL
- U5 pad 2: unconnected-(U5-GND-Pad2) -> GND
- U5 pad 3: unconnected-(U5-ALERT-Pad3) -> TMP102_ALERT
- U5 pad 4: unconnected-(U5-ADD0-Pad4) -> GND
- U5 pad 5: unconnected-(U5-V+-Pad5) -> EXT_VCC
- U5 pad 6: unconnected-(U5-SDA-Pad6) -> SDA
Routing:
- added copper zone on In2.Cu, net EXT_VCC
- added copper zone on In1.Cu, net GND
- added copper zone on In2.Cu, net VBAT
Other:
- board text added: "1"
- board text added: "2"
- board text added: "C"
- board text added: "D"
- board text added: "SWCLK"
- board text added: "SWD"
- board text removed: "B+"
- board text removed: "B-"
- board text removed: "U4"

Commit message: added caps
Parts:
- removed the R1 at (168.3, 100.4)
- added C10: CC0402KRX7R7BB104, easyeda2kicad:C0402, F.Cu at (160.8, 105.7)
- added C11: CC0402KRX7R7BB104, easyeda2kicad:C0402, F.Cu at (160.1, 117.9)
- added C12: CC0402KRX7R7BB104, easyeda2kicad:C0402, F.Cu at (162.4, 114.0)
- added C13: CC0603JRNPO8BN561, easyeda2kicad:C0603, F.Cu at (162.7, 117.2)
- added C14: CC0603JRNPO8BN561, easyeda2kicad:C0603, F.Cu at (164.7, 117.2)
- added C2: CL21A106KAYNNNE, easyeda2kicad:C0805, F.Cu at (165.8, 114.3)
- added C4: CL31A107MQHNNNE, easyeda2kicad:C1206, F.Cu at (162.7, 101.3)
- added C5: CL31A107MQHNNNE, easyeda2kicad:C1206, F.Cu at (169.1, 101.2)
- added C6: CL31A107MQHNNNE, easyeda2kicad:C1206, F.Cu at (166.7, 101.1)
- added C7: CL31A107MQHNNNE, easyeda2kicad:C1206, F.Cu at (160.1, 101.3)
- added C8: CC0402KRX7R7BB104, easyeda2kicad:C0402, F.Cu at (158.1, 100.0)
- added C9: CC0402KRX7R7BB104, easyeda2kicad:C0402, F.Cu at (169.3, 89.9)
- moved TP1 18.5 mm to (183.0, 115.6)
- moved TP4 17.0 mm to (183.0, 112.0)
- moved TP3 13.4 mm to (182.6, 117.5)
- moved R1 10.6 mm to (167.8, 104.8)
- moved R2 4.44 mm to (169.9, 104.8)
- moved U1 1.50 mm to (163.9, 110.9)
- moved U5 0.54 mm to (168.4, 121.3)
- moved U4 0.10 mm to (166.9, 94.7)
- moved U6 0.10 mm to (160.9, 94.7)
- moved H1 0.07 mm to (170.5, 87.4)
- moved H2 0.07 mm to (157.0, 87.4)
- moved H3 0.07 mm to (163.8, 89.7)
Connections:
- net /P0.09 renamed NFC1
- net /P0.10 renamed NFC2
- H3 pad 1: Net-(U6-Bout) -> Net-(U6-Aout)
- H3 pad 2: Net-(U6-Aout) -> Net-(U6-Bout)
- H3 pad 3: Net-(U4-Bout) -> Net-(U4-Aout)
- H3 pad 4: Net-(U4-Aout) -> Net-(U4-Bout)
- SW2 pad 3: unconnected-(SW2-Pad3) -> GND
- SW2 pad 4: unconnected-(SW2-Pad4) -> RESET
- U1 pad 2: unconnected-(U1-VCC-Pad2) -> Net-(U1-VCC)
- U4 pad 1: unconnected-(U4-Vcc-Pad1) -> Net-(U4-Vcc)
- U6 pad 1: unconnected-(U6-Vcc-Pad1) -> Net-(U6-Vcc)
Other:
- outline, holes or cut-outs redrawn

Commit message: midway through routing LED matrix
Parts:
- added C1: CL10B224KA8NNNC, easyeda2kicad:C0603, F.Cu at (166.9, 107.3)
- added JP1: Jumper_3_Bridged12, Jumper:SolderJumper-3_P1.3mm_Bridged12_Pad1.0x1.5mm_NumberLabels, F.Cu at (163.9, 86.8)
- added TP8: AUDIO-IN, TestPoint:TestPoint_Pad_D1.0mm, F.Cu at (169.3, 107.3)
- moved LED71 7.40 mm to (169.2, 110.0), turned to -45 degrees
- moved LED72 7.40 mm to (167.4, 110.0), turned to -45 degrees
- moved LED73 7.40 mm to (165.6, 110.0), turned to -45 degrees
- moved LED74 7.40 mm to (163.8, 110.0), turned to -45 degrees
- moved LED75 7.40 mm to (162.0, 110.0), turned to -45 degrees
- moved LED76 7.40 mm to (160.2, 110.0), turned to -45 degrees
- moved LED77 7.40 mm to (158.4, 110.0), turned to -45 degrees
- moved LEDC1-R6 7.16 mm to (158.4, 101.2), turned to -45 degrees
- moved LEDC2-R6 7.16 mm to (160.2, 101.2), turned to -45 degrees
- moved LEDC3-R6 7.16 mm to (162.0, 101.2), turned to -45 degrees
- moved LEDC4-R6 7.16 mm to (163.8, 101.2), turned to -45 degrees
- moved LEDC5-R6 7.16 mm to (165.6, 101.2), turned to -45 degrees
- moved LEDC6-R6 7.16 mm to (167.4, 101.2), turned to -45 degrees
- moved LEDC7-R6 7.16 mm to (169.2, 101.2), turned to -45 degrees
- moved LED64 7.11 mm to (169.2, 108.3), turned to -45 degrees
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- renumbered LED7 to LEDC1-R1, LED14 to LEDC1-R2, LED21 to LEDC1-R3, LED28 to LEDC1-R4, LED35 to LEDC1-R5, LED42 to LEDC1-R6, LED49 to LEDC1-R7, LED56 to LEDC1-R8, LED6 to LEDC2-R1, LED13 to LEDC2-R2, LED20 to LEDC2-R3, LED27 to LEDC2-R4, LED34 to LEDC2-R5, LED41 to LEDC2-R6, LED48 to LEDC2-R7, LED55 to LEDC2-R8, LED5 to LEDC3-R1, LED12 to LEDC3-R2, LED19 to LEDC3-R3, LED26 to LEDC3-R4, LED33 to LEDC3-R5, LED40 to LEDC3-R6, LED47 to LEDC3-R7, LED54 to LEDC3-R8, LED4 to LEDC4-R1, LED11 to LEDC4-R2, LED18 to LEDC4-R3, LED25 to LEDC4-R4, LED32 to LEDC4-R5, LED39 to LEDC4-R6, LED46 to LEDC4-R7, LED53 to LEDC4-R8, LED3 to LEDC5-R1, LED10 to LEDC5-R2, LED17 to LEDC5-R3, LED24 to LEDC5-R4, LED31 to LEDC5-R5, LED38 to LEDC5-R6, LED45 to LEDC5-R7, LED52 to LEDC5-R8, LED2 to LEDC6-R1, LED9 to LEDC6-R2, LED16 to LEDC6-R3, LED23 to LEDC6-R4, LED30 to LEDC6-R5, LED37 to LEDC6-R6, LED44 to LEDC6-R7, LED51 to LEDC6-R8, LED1 to LEDC7-R1, LED8 to LEDC7-R2, LED15 to LEDC7-R3, LED22 to LEDC7-R4, LED29 to LEDC7-R5, LED36 to LEDC7-R6, LED43 to LEDC7-R7, LED50 to LEDC7-R8
Connections:
- C4 pad 2: Net-(U6-Vcc) -> MOTOR-PWR
- C5 pad 2: Net-(U4-Vcc) -> MOTOR-PWR
- C6 pad 2: Net-(U4-Vcc) -> MOTOR-PWR
- C7 pad 2: Net-(U6-Vcc) -> MOTOR-PWR
- C8 pad 2: Net-(U6-Vcc) -> MOTOR-PWR
- C9 pad 2: Net-(U4-Vcc) -> MOTOR-PWR
- LEDC1-R1 pad 1: unconnected-(LED7-K-Pad1) -> /CA1
- LEDC1-R1 pad 2: unconnected-(LED7-A-Pad2) -> /CA2
- LEDC1-R2 pad 1: unconnected-(LED14-K-Pad1) -> /CA1
- LEDC1-R2 pad 2: unconnected-(LED14-A-Pad2) -> /CA3
- LEDC1-R3 pad 1: unconnected-(LED21-K-Pad1) -> /CA1
- LEDC1-R3 pad 2: unconnected-(LED21-A-Pad2) -> /CA4
- LEDC1-R4 pad 1: unconnected-(LED28-K-Pad1) -> /CA1
- LEDC1-R4 pad 2: unconnected-(LED28-A-Pad2) -> /CA5
- LEDC1-R5 pad 1: unconnected-(LED35-K-Pad1) -> /CA1
- LEDC1-R5 pad 2: unconnected-(LED35-A-Pad2) -> /CA6
- LEDC1-R6 pad 1: unconnected-(LED42-K-Pad1) -> /CA1
- LEDC1-R6 pad 2: unconnected-(LED42-A-Pad2) -> /CA7
- LEDC1-R7 pad 1: unconnected-(LED49-K-Pad1) -> /CA1
- LEDC1-R7 pad 2: unconnected-(LED49-A-Pad2) -> /CA8
- LEDC1-R8 pad 1: unconnected-(LED56-K-Pad1) -> /CA1
- LEDC1-R8 pad 2: unconnected-(LED56-A-Pad2) -> /CA9
- LEDC2-R1 pad 1: unconnected-(LED6-K-Pad1) -> /CA2
- LEDC2-R1 pad 2: unconnected-(LED6-A-Pad2) -> /CA1
- LEDC2-R2 pad 1: unconnected-(LED13-K-Pad1) -> /CA2
- LEDC2-R2 pad 2: unconnected-(LED13-A-Pad2) -> /CA3
- LEDC2-R3 pad 1: unconnected-(LED20-K-Pad1) -> /CA2
- LEDC2-R3 pad 2: unconnected-(LED20-A-Pad2) -> /CA4
- LEDC2-R4 pad 1: unconnected-(LED27-K-Pad1) -> /CA2
- LEDC2-R4 pad 2: unconnected-(LED27-A-Pad2) -> /CA5
- LEDC2-R5 pad 1: unconnected-(LED34-K-Pad1) -> /CA2
- LEDC2-R5 pad 2: unconnected-(LED34-A-Pad2) -> /CA6
- LEDC2-R6 pad 1: unconnected-(LED41-K-Pad1) -> /CA2
- LEDC2-R6 pad 2: unconnected-(LED41-A-Pad2) -> /CA7
- LEDC2-R7 pad 1: unconnected-(LED48-K-Pad1) -> /CA2
- LEDC2-R7 pad 2: unconnected-(LED48-A-Pad2) -> /CA8
- LEDC2-R8 pad 1: unconnected-(LED55-K-Pad1) -> /CA2
- LEDC2-R8 pad 2: unconnected-(LED55-A-Pad2) -> /CA9
- LEDC3-R1 pad 1: unconnected-(LED5-K-Pad1) -> /CA3
- LEDC3-R1 pad 2: unconnected-(LED5-A-Pad2) -> /CA1
- LEDC3-R2 pad 1: unconnected-(LED12-K-Pad1) -> /CA3
- LEDC3-R2 pad 2: unconnected-(LED12-A-Pad2) -> /CA2
- LEDC3-R3 pad 1: unconnected-(LED19-K-Pad1) -> /CA3
- LEDC3-R3 pad 2: unconnected-(LED19-A-Pad2) -> /CA4
- LEDC3-R4 pad 1: unconnected-(LED26-K-Pad1) -> /CA3
- LEDC3-R4 pad 2: unconnected-(LED26-A-Pad2) -> /CA5
- LEDC3-R5 pad 1: unconnected-(LED33-K-Pad1) -> /CA3
- LEDC3-R5 pad 2: unconnected-(LED33-A-Pad2) -> /CA6
- LEDC3-R6 pad 1: unconnected-(LED40-K-Pad1) -> /CA3
- LEDC3-R6 pad 2: unconnected-(LED40-A-Pad2) -> /CA7
- LEDC3-R7 pad 1: unconnected-(LED47-K-Pad1) -> /CA3
- LEDC3-R7 pad 2: unconnected-(LED47-A-Pad2) -> /CA8
- LEDC3-R8 pad 1: unconnected-(LED54-K-Pad1) -> /CA3
- LEDC3-R8 pad 2: unconnected-(LED54-A-Pad2) -> /CA9
- LEDC4-R1 pad 1: unconnected-(LED4-K-Pad1) -> /CA4
- LEDC4-R1 pad 2: unconnected-(LED4-A-Pad2) -> /CA1
- LEDC4-R2 pad 1: unconnected-(LED11-K-Pad1) -> /CA4
- LEDC4-R2 pad 2: unconnected-(LED11-A-Pad2) -> /CA2
- LEDC4-R3 pad 1: unconnected-(LED18-K-Pad1) -> /CA4
- LEDC4-R3 pad 2: unconnected-(LED18-A-Pad2) -> /CA3
- LEDC4-R4 pad 1: unconnected-(LED25-K-Pad1) -> /CA4
- LEDC4-R4 pad 2: unconnected-(LED25-A-Pad2) -> /CA5
- LEDC4-R5 pad 1: unconnected-(LED32-K-Pad1) -> /CA4
- LEDC4-R5 pad 2: unconnected-(LED32-A-Pad2) -> /CA6
- LEDC4-R6 pad 1: unconnected-(LED39-K-Pad1) -> /CA4
- LEDC4-R6 pad 2: unconnected-(LED39-A-Pad2) -> /CA7
- LEDC4-R7 pad 1: unconnected-(LED46-K-Pad1) -> /CA4
- LEDC4-R7 pad 2: unconnected-(LED46-A-Pad2) -> /CA8
- LEDC4-R8 pad 1: unconnected-(LED53-K-Pad1) -> /CA4
- LEDC4-R8 pad 2: unconnected-(LED53-A-Pad2) -> /CA9
- LEDC5-R1 pad 1: unconnected-(LED3-K-Pad1) -> /CA5
- LEDC5-R1 pad 2: unconnected-(LED3-A-Pad2) -> /CA1
- LEDC5-R2 pad 1: unconnected-(LED10-K-Pad1) -> /CA5
- LEDC5-R2 pad 2: unconnected-(LED10-A-Pad2) -> /CA2
- LEDC5-R3 pad 1: unconnected-(LED17-K-Pad1) -> /CA5
- LEDC5-R3 pad 2: unconnected-(LED17-A-Pad2) -> /CA3
- LEDC5-R4 pad 1: unconnected-(LED24-K-Pad1) -> /CA5
- LEDC5-R4 pad 2: unconnected-(LED24-A-Pad2) -> /CA4
- LEDC5-R5 pad 1: unconnected-(LED31-K-Pad1) -> /CA5
- LEDC5-R5 pad 2: unconnected-(LED31-A-Pad2) -> /CA6
- LEDC5-R6 pad 1: unconnected-(LED38-K-Pad1) -> /CA5
- LEDC5-R6 pad 2: unconnected-(LED38-A-Pad2) -> /CA7
- LEDC5-R7 pad 1: unconnected-(LED45-K-Pad1) -> /CA5
- LEDC5-R7 pad 2: unconnected-(LED45-A-Pad2) -> /CA8
- LEDC5-R8 pad 1: unconnected-(LED52-K-Pad1) -> /CA5
- LEDC5-R8 pad 2: unconnected-(LED52-A-Pad2) -> /CA9
- LEDC6-R1 pad 1: unconnected-(LED2-K-Pad1) -> /CA6
- LEDC6-R1 pad 2: unconnected-(LED2-A-Pad2) -> /CA1
- LEDC6-R2 pad 1: unconnected-(LED9-K-Pad1) -> /CA6
- LEDC6-R2 pad 2: unconnected-(LED9-A-Pad2) -> /CA2
- LEDC6-R3 pad 1: unconnected-(LED16-K-Pad1) -> /CA6
- LEDC6-R3 pad 2: unconnected-(LED16-A-Pad2) -> /CA3
- LEDC6-R4 pad 1: unconnected-(LED23-K-Pad1) -> /CA6
- LEDC6-R4 pad 2: unconnected-(LED23-A-Pad2) -> /CA4
- LEDC6-R5 pad 1: unconnected-(LED30-K-Pad1) -> /CA6
- LEDC6-R5 pad 2: unconnected-(LED30-A-Pad2) -> /CA5
- LEDC6-R6 pad 1: unconnected-(LED37-K-Pad1) -> /CA6
- LEDC6-R6 pad 2: unconnected-(LED37-A-Pad2) -> /CA7
- LEDC6-R7 pad 1: unconnected-(LED44-K-Pad1) -> /CA6
- LEDC6-R7 pad 2: unconnected-(LED44-A-Pad2) -> /CA8
- LEDC6-R8 pad 1: unconnected-(LED51-K-Pad1) -> /CA6
- LEDC6-R8 pad 2: unconnected-(LED51-A-Pad2) -> /CA9
- LEDC7-R1 pad 1: unconnected-(LED1-K-Pad1) -> /CA7
- LEDC7-R1 pad 2: unconnected-(LED1-A-Pad2) -> /CA1
- LEDC7-R2 pad 1: unconnected-(LED8-K-Pad1) -> /CA7
- LEDC7-R2 pad 2: unconnected-(LED8-A-Pad2) -> /CA2
- LEDC7-R3 pad 1: unconnected-(LED15-K-Pad1) -> /CA7
- LEDC7-R3 pad 2: unconnected-(LED15-A-Pad2) -> /CA3
- LEDC7-R4 pad 1: unconnected-(LED22-K-Pad1) -> /CA7
- LEDC7-R4 pad 2: unconnected-(LED22-A-Pad2) -> /CA4
- LEDC7-R5 pad 1: unconnected-(LED29-K-Pad1) -> /CA7
- LEDC7-R5 pad 2: unconnected-(LED29-A-Pad2) -> /CA5
- LEDC7-R6 pad 1: unconnected-(LED36-K-Pad1) -> /CA7
- LEDC7-R6 pad 2: unconnected-(LED36-A-Pad2) -> /CA6
- LEDC7-R7 pad 1: unconnected-(LED43-K-Pad1) -> /CA7
- LEDC7-R7 pad 2: unconnected-(LED43-A-Pad2) -> /CA8
- LEDC7-R8 pad 1: unconnected-(LED50-K-Pad1) -> /CA7
- LEDC7-R8 pad 2: unconnected-(LED50-A-Pad2) -> /CA9
- U1 pad 17: unconnected-(U1-IN-Pad17) -> Net-(U1-IN)
- U1 pad 19: unconnected-(U1-SDA-Pad19) -> SDA
- U1 pad 20: unconnected-(U1-SCL-Pad20) -> SCL
- U4 pad 1: Net-(U4-Vcc) -> MOTOR-PWR
- U4 pad 4: unconnected-(U4-GND-Pad4) -> GND
- U4 pad 7: unconnected-(U4-GND-Pad7) -> GND
- U6 pad 1: Net-(U6-Vcc) -> MOTOR-PWR
- U6 pad 4: unconnected-(U6-GND-Pad4) -> GND
- U6 pad 7: unconnected-(U6-GND-Pad7) -> GND
Routing:
- net /CA1: track 0.00 -> 34.2 mm
- net /CA6: track 0.00 -> 28.5 mm, vias 0 -> 7
- net /CA5: track 0.00 -> 27.7 mm, vias 0 -> 6
- net /CA4: track 0.00 -> 26.4 mm, vias 0 -> 7
- net RESET: track 0.00 -> 26.1 mm, vias 0 -> 1
- net /CA3: track 0.00 -> 25.7 mm, vias 0 -> 7
- net /CA2: track 0.00 -> 24.3 mm, vias 0 -> 6
- net /CA7: track 0.00 -> 23.3 mm, vias 0 -> 6
- net MOTOR2-A: track 0.00 -> 20.8 mm, vias 0 -> 2
- net MOTOR2-B: track 0.00 -> 18.1 mm, vias 0 -> 3
- net VBAT: track 0.00 -> 17.2 mm, vias 0 -> 4
- net MOTOR1-A: track 0.00 -> 12.9 mm, vias 0 -> 2
- net /CA8: track 0.00 -> 11.0 mm, vias 0 -> 5
- net /CA9: track 0.00 -> 10.8 mm
- net GND: track 0.00 -> 10.5 mm, vias 0 -> 16
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- added copper zone on F.Cu, net MOTOR-PWR
- added copper zone on In2.Cu, net MOTOR-PWR

Commit message: all connections to LEDs made on schematics
Parts:
- renumbered LED70 to LEDC1-R10, LED77 to LEDC1-R11, LED84 to LEDC1-R12, LED91 to LEDC1-R13, LED98 to LEDC1-R14, LED105 to LEDC1-R15, LED63 to LEDC1-R9, LED69 to LEDC2-R10, LED76 to LEDC2-R11, LED83 to LEDC2-R12, LED90 to LEDC2-R13, LED97 to LEDC2-R14, LED104 to LEDC2-R15, LED62 to LEDC2-R9, LED68 to LEDC3-R10, LED75 to LEDC3-R11, LED82 to LEDC3-R12, LED89 to LEDC3-R13, LED96 to LEDC3-R14, LED103 to LEDC3-R15, LED61 to LEDC3-R9, LED67 to LEDC4-R10, LED74 to LEDC4-R11, LED81 to LEDC4-R12, LED88 to LEDC4-R13, LED95 to LEDC4-R14, LED102 to LEDC4-R15, LED60 to LEDC4-R9, LED66 to LEDC5-R10, LED73 to LEDC5-R11, LED80 to LEDC5-R12, LED87 to LEDC5-R13, LED94 to LEDC5-R14, LED101 to LEDC5-R15, LED59 to LEDC5-R9, LED65 to LEDC6-R10, LED72 to LEDC6-R11, LED79 to LEDC6-R12, LED86 to LEDC6-R13, LED93 to LEDC6-R14, LED100 to LEDC6-R15, LED58 to LEDC6-R9, LED64 to LEDC7-R10, LED71 to LEDC7-R11, LED78 to LEDC7-R12, LED85 to LEDC7-R13, LED92 to LEDC7-R14, LED99 to LEDC7-R15, LED57 to LEDC7-R9
Connections:
- LEDC1-R10 pad 1: unconnected-(LED70-K-Pad1) -> /CB1
- LEDC1-R10 pad 2: unconnected-(LED70-A-Pad2) -> /CB3
- LEDC1-R11 pad 1: unconnected-(LED77-K-Pad1) -> /CB1
- LEDC1-R11 pad 2: unconnected-(LED77-A-Pad2) -> /CB4
- LEDC1-R12 pad 1: unconnected-(LED84-K-Pad1) -> /CB1
- LEDC1-R12 pad 2: unconnected-(LED84-A-Pad2) -> /CB5
- LEDC1-R13 pad 1: unconnected-(LED91-K-Pad1) -> /CB1
- LEDC1-R13 pad 2: unconnected-(LED91-A-Pad2) -> /CB6
- LEDC1-R14 pad 1: unconnected-(LED98-K-Pad1) -> /CB1
- LEDC1-R14 pad 2: unconnected-(LED98-A-Pad2) -> /CB7
- LEDC1-R15 pad 1: unconnected-(LED105-K-Pad1) -> /CB1
- LEDC1-R15 pad 2: unconnected-(LED105-A-Pad2) -> /CB8
- LEDC1-R9 pad 1: unconnected-(LED63-K-Pad1) -> /CB1
- LEDC1-R9 pad 2: unconnected-(LED63-A-Pad2) -> /CB2
- LEDC2-R10 pad 1: unconnected-(LED69-K-Pad1) -> /CB2
- LEDC2-R10 pad 2: unconnected-(LED69-A-Pad2) -> /CB3
- LEDC2-R11 pad 1: unconnected-(LED76-K-Pad1) -> /CB2
- LEDC2-R11 pad 2: unconnected-(LED76-A-Pad2) -> /CB4
- LEDC2-R12 pad 1: unconnected-(LED83-K-Pad1) -> /CB2
- LEDC2-R12 pad 2: unconnected-(LED83-A-Pad2) -> /CB5
- LEDC2-R13 pad 1: unconnected-(LED90-K-Pad1) -> /CB2
- LEDC2-R13 pad 2: unconnected-(LED90-A-Pad2) -> /CB6
- LEDC2-R14 pad 1: unconnected-(LED97-K-Pad1) -> /CB2
- LEDC2-R14 pad 2: unconnected-(LED97-A-Pad2) -> /CB7
- LEDC2-R15 pad 1: unconnected-(LED104-K-Pad1) -> /CB2
- LEDC2-R15 pad 2: unconnected-(LED104-A-Pad2) -> /CB8
- LEDC2-R9 pad 1: unconnected-(LED62-K-Pad1) -> /CB2
- LEDC2-R9 pad 2: unconnected-(LED62-A-Pad2) -> /CB1
- LEDC3-R10 pad 1: unconnected-(LED68-K-Pad1) -> /CB3
- LEDC3-R10 pad 2: unconnected-(LED68-A-Pad2) -> /CB2
- LEDC3-R11 pad 1: unconnected-(LED75-K-Pad1) -> /CB3
- LEDC3-R11 pad 2: unconnected-(LED75-A-Pad2) -> /CB4
- LEDC3-R12 pad 1: unconnected-(LED82-K-Pad1) -> /CB3
- LEDC3-R12 pad 2: unconnected-(LED82-A-Pad2) -> /CB5
- LEDC3-R13 pad 1: unconnected-(LED89-K-Pad1) -> /CB3
- LEDC3-R13 pad 2: unconnected-(LED89-A-Pad2) -> /CB6
- LEDC3-R14 pad 1: unconnected-(LED96-K-Pad1) -> /CB3
- LEDC3-R14 pad 2: unconnected-(LED96-A-Pad2) -> /CB7
- LEDC3-R15 pad 1: unconnected-(LED103-K-Pad1) -> /CB3
- LEDC3-R15 pad 2: unconnected-(LED103-A-Pad2) -> /CB8
- LEDC3-R9 pad 1: unconnected-(LED61-K-Pad1) -> /CB3
- LEDC3-R9 pad 2: unconnected-(LED61-A-Pad2) -> /CB1
- LEDC4-R10 pad 1: unconnected-(LED67-K-Pad1) -> /CB4
- LEDC4-R10 pad 2: unconnected-(LED67-A-Pad2) -> /CB2
- LEDC4-R11 pad 1: unconnected-(LED74-K-Pad1) -> /CB4
- LEDC4-R11 pad 2: unconnected-(LED74-A-Pad2) -> /CB3
- LEDC4-R12 pad 1: unconnected-(LED81-K-Pad1) -> /CB4
- LEDC4-R12 pad 2: unconnected-(LED81-A-Pad2) -> /CB5
- LEDC4-R13 pad 1: unconnected-(LED88-K-Pad1) -> /CB4
- LEDC4-R13 pad 2: unconnected-(LED88-A-Pad2) -> /CB6
- LEDC4-R14 pad 1: unconnected-(LED95-K-Pad1) -> /CB4
- LEDC4-R14 pad 2: unconnected-(LED95-A-Pad2) -> /CB7
- LEDC4-R15 pad 1: unconnected-(LED102-K-Pad1) -> /CB4
- LEDC4-R15 pad 2: unconnected-(LED102-A-Pad2) -> /CB8
- LEDC4-R9 pad 1: unconnected-(LED60-K-Pad1) -> /CB4
- LEDC4-R9 pad 2: unconnected-(LED60-A-Pad2) -> /CB1
- LEDC5-R10 pad 1: unconnected-(LED66-K-Pad1) -> /CB5
- LEDC5-R10 pad 2: unconnected-(LED66-A-Pad2) -> /CB2
- LEDC5-R11 pad 1: unconnected-(LED73-K-Pad1) -> /CB5
- LEDC5-R11 pad 2: unconnected-(LED73-A-Pad2) -> /CB3
- LEDC5-R12 pad 1: unconnected-(LED80-K-Pad1) -> /CB5
- LEDC5-R12 pad 2: unconnected-(LED80-A-Pad2) -> /CB4
- LEDC5-R13 pad 1: unconnected-(LED87-K-Pad1) -> /CB5
- LEDC5-R13 pad 2: unconnected-(LED87-A-Pad2) -> /CB6
- LEDC5-R14 pad 1: unconnected-(LED94-K-Pad1) -> /CB5
- LEDC5-R14 pad 2: unconnected-(LED94-A-Pad2) -> /CB7
- LEDC5-R15 pad 1: unconnected-(LED101-K-Pad1) -> /CB5
- LEDC5-R15 pad 2: unconnected-(LED101-A-Pad2) -> /CB8
- LEDC5-R9 pad 1: unconnected-(LED59-K-Pad1) -> /CB5
- LEDC5-R9 pad 2: unconnected-(LED59-A-Pad2) -> /CB1
- LEDC6-R10 pad 1: unconnected-(LED65-K-Pad1) -> /CB6
- LEDC6-R10 pad 2: unconnected-(LED65-A-Pad2) -> /CB2
- LEDC6-R11 pad 1: unconnected-(LED72-K-Pad1) -> /CB6
- LEDC6-R11 pad 2: unconnected-(LED72-A-Pad2) -> /CB3
- LEDC6-R12 pad 1: unconnected-(LED79-K-Pad1) -> /CB6
- LEDC6-R12 pad 2: unconnected-(LED79-A-Pad2) -> /CB4
- LEDC6-R13 pad 1: unconnected-(LED86-K-Pad1) -> /CB6
- LEDC6-R13 pad 2: unconnected-(LED86-A-Pad2) -> /CB5
- LEDC6-R14 pad 1: unconnected-(LED93-K-Pad1) -> /CB6
- LEDC6-R14 pad 2: unconnected-(LED93-A-Pad2) -> /CB7
- LEDC6-R15 pad 1: unconnected-(LED100-K-Pad1) -> /CB6
- LEDC6-R15 pad 2: unconnected-(LED100-A-Pad2) -> /CB8
- LEDC6-R9 pad 1: unconnected-(LED58-K-Pad1) -> /CB6
- LEDC6-R9 pad 2: unconnected-(LED58-A-Pad2) -> /CB1
- LEDC7-R10 pad 1: unconnected-(LED64-K-Pad1) -> /CB7
- LEDC7-R10 pad 2: unconnected-(LED64-A-Pad2) -> /CB2
- LEDC7-R11 pad 1: unconnected-(LED71-K-Pad1) -> /CB7
- LEDC7-R11 pad 2: unconnected-(LED71-A-Pad2) -> /CB3
- LEDC7-R12 pad 1: unconnected-(LED78-K-Pad1) -> /CB7
- LEDC7-R12 pad 2: unconnected-(LED78-A-Pad2) -> /CB4
- LEDC7-R13 pad 1: unconnected-(LED85-K-Pad1) -> /CB7
- LEDC7-R13 pad 2: unconnected-(LED85-A-Pad2) -> /CB5
- LEDC7-R14 pad 1: unconnected-(LED92-K-Pad1) -> /CB7
- LEDC7-R14 pad 2: unconnected-(LED92-A-Pad2) -> /CB6
- LEDC7-R15 pad 1: unconnected-(LED99-K-Pad1) -> /CB7
- LEDC7-R15 pad 2: unconnected-(LED99-A-Pad2) -> /CB8
- LEDC7-R9 pad 1: unconnected-(LED57-K-Pad1) -> /CB7
- LEDC7-R9 pad 2: unconnected-(LED57-A-Pad2) -> /CB1
- U1 pad 1: unconnected-(U1-CA9-Pad1) -> /CA9
- U1 pad 10: unconnected-(U1-CB4-Pad10) -> /CB4
- U1 pad 11: unconnected-(U1-CB5-Pad11) -> /CB5
- U1 pad 12: unconnected-(U1-CB6-Pad12) -> /CB6
- U1 pad 13: unconnected-(U1-CB7-Pad13) -> /CB7
- U1 pad 14: unconnected-(U1-CB8-Pad14) -> /CB8
- U1 pad 15: unconnected-(U1-CB9-Pad15) -> /CB9
- U1 pad 21: unconnected-(U1-CA1-Pad21) -> /CA1
- U1 pad 22: unconnected-(U1-CA2-Pad22) -> /CA2
- U1 pad 23: unconnected-(U1-CA3-Pad23) -> /CA3
- U1 pad 24: unconnected-(U1-CA4-Pad24) -> /CA4
- U1 pad 25: unconnected-(U1-CA5-Pad25) -> /CA5
- U1 pad 26: unconnected-(U1-CA6-Pad26) -> /CA6
- U1 pad 27: unconnected-(U1-CA7-Pad27) -> /CA7
- U1 pad 28: unconnected-(U1-CA8-Pad28) -> /CA8
- U1 pad 3: unconnected-(U1-SDB-Pad3) -> LED_SDB
- U1 pad 4: unconnected-(U1-INTB-Pad4) -> LED_INT
- U1 pad 5: unconnected-(U1-GND-Pad5) -> GND
- U1 pad 7: unconnected-(U1-CB1-Pad7) -> /CB1
- U1 pad 8: unconnected-(U1-CB2-Pad8) -> /CB2
- U1 pad 9: unconnected-(U1-CB3-Pad9) -> /CB3
Routing:
- net /CB6: track 0.00 -> 10.4 mm
- net /CB1: track 0.00 -> 10.4 mm
- net /CB5: track 0.00 -> 10.4 mm
- net /CB4: track 0.00 -> 10.4 mm
- net /CB3: track 0.00 -> 10.4 mm
- net /CB7: track 0.00 -> 10.4 mm
- net /CB2: track 0.00 -> 10.4 mm
- net /CA7: track 23.3 -> 28.4 mm
