File: tikk-hw.kicad_pcb (KiCad board)
At the start: 4 copper layers, 18.1 x 39 mm, 155 parts, among them J1 51281-0598, P6 ZX-SH1.0-4PWT, SW1 TS24CA, SW2 TS24CA, U1 IS31FL3731-QFLS2-TR, U2 LIS2DH12TR, U3 Tenstar nRF52840, U4 CP6208DTR(XBLW), U5 TMP102AIDRLR, U6 CP6208DTR(XBLW)

Commit message: final changes before sending to JLC
Parts:
- removed U6: CP6208DTR(XBLW), easyeda2kicad:SOP-8_L4.9-W3.9-P1.27-LS6.0-BL
- added U7: L9110S_C5157607, easyeda2kicad:SOP-8_L4.9-W3.9-P1.27-LS6.0-BL, F.Cu at (160.9, 94.7)
- U4: value CP6208DTR(XBLW) -> L9110S_C5157607
- moved C2 0.20 mm to (165.8, 114.5)
Connections:
- H3 pad 3: Net-(U4-Aout) -> Net-(U4-OB)
- H3 pad 4: Net-(U4-Bout) -> Net-(U4-OA)
- U3 pad 8: /P1.15 -> LED_INT
- U3 pad 9: /P1.13 -> LED_SDB
- U4 pad 1: MOTOR-PWR -> Net-(U4-OA)
- U4 pad 2: Net-(U4-Bout) -> MOTOR-PWR
- U4 pad 3: Net-(U4-Aout) -> MOTOR-PWR
- U4 pad 4: GND -> Net-(U4-OB)
- U4 pad 5: MOTOR2-B -> GND
- U4 pad 6: unconnected-(U4-NC-Pad6) -> MOTOR2-A
- U4 pad 7: GND -> MOTOR2-B
- U4 pad 8: MOTOR2-A -> GND
Routing:
- net LED_INT: track 0.00 -> 18.2 mm, vias 0 -> 2
- net LED_SDB: track 0.00 -> 15.8 mm, vias 0 -> 1
- net /CB4: track 26.3 -> 31.4 mm, vias 6 -> 5
- net GND: track 42.0 -> 37.8 mm, vias 70 -> 68
- net MOTOR1-A: track 12.7 -> 16.9 mm
- net Net-(U4-Aout): track 3.11 -> 0.00 mm
- net Net-(U4-OA): track 0.00 -> 2.89 mm
- net Net-(U4-OB): track 0.00 -> 2.80 mm
- net MOTOR2-B: track 16.3 -> 19.0 mm
- net MOTOR1-B: track 4.05 -> 6.57 mm, vias 1 -> 0
- net Net-(U4-Bout): track 2.34 -> 0.00 mm
- net MOTOR2-A: track 21.9 -> 23.9 mm, vias 2 -> 3
- net /CB6: track 29.8 -> 31.5 mm
- net EXT_VCC: track 16.7 -> 15.7 mm, vias 11 -> 12
- net /CA4: track 34.9 -> 34.1 mm
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