File: tikk-hw.kicad_sch (KiCad schematic)
At the start: 155 parts, among them J1 51281-0598, P6 ZX-SH1.0-4PWT, SW1 TS24CA, SW2 TS24CA, U1 IS31FL3731-QFLS2-TR, U2 LIS2DH12TR, U3 Tenstar nRF52840, U4 CP6208DTR(XBLW), U5 TMP102AIDRLR, U6 CP6208DTR(XBLW)

Commit message: final changes before sending to JLC
Parts:
- removed U4, U6: CP6208DTR(XBLW), easyeda2kicad:SOP-8_L4.9-W3.9-P1.27-LS6.0-BL, symbol easyeda2kicad:CP6208DTR(XBLW)
- added U4, U7: L9110S_C5157607, easyeda2kicad:SOP-8_L4.9-W3.9-P1.27-LS6.0-BL, symbol easyeda2kicad:L9110S_C5157607
Connections:
- net P1.13 is gone; now on net LED_SDB: U3.9 (1.13)
- net P1.15 is gone; now on net LED_INT: U3.8 (1.15)
- net GND: now also U4.5 (GND), U4.8 (GND), U7.5 (GND), U7.8 (GND)
- net MOTOR-PWR: now also U4.2 (VCC), U4.3 (VCC), U7.2 (VCC), U7.3 (VCC)
- net MOTOR1-A: now also U7.6 (IA)
- net MOTOR1-B: now also U7.7 (IB)
- net MOTOR2-A: now also U4.6 (IA)
- net MOTOR2-B: now also U4.7 (IB)
- net at H3.2: now also U7.1 (OA)
- net at H3.1: now also U7.4 (OB)
- net at H3.4: now also U4.1 (OA)
- net at H3.3: now also U4.4 (OB)
- no-connect marks 9 -> 5
