File: tikk-hw.kicad_sch (KiCad schematic)
At the start: 155 parts, among them J1 51281-0598, P6 ZX-SH1.0-4PWT, SW1 TS24CA, SW2 TS24CA, U1 IS31FL3731-QFLS2-TR, U2 LIS2DH12TR, U3 Tenstar nRF52840, U4 L9110S_C5157607, U5 TMP102AIDRLR, U7 L9110S_C5157607

Commit message: Clean up repo before open sourcing, pull in final data changes on schematic
Parts:
- H3: now fitted
Changed lines of the file:
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@@
 		(in_bom yes)
 		(on_board yes)
-		(dnp yes)
+		(dnp no)
 		(property "Reference" "H3"
 			(at 419.1 204.4699 0)
